File: kicad/customBoard/customBoard.kicad_sch (KiCad schematic)
At the start: 0 parts

Commit message: First draft of the power circuit
While this is my first time developing any kind of PCB, this circuit is pretty similar to an existing schematic, so it should be pretty solid.
Other:
- added sheet power (power.kicad_sch)
