File: kicad/customBoard/customBoard.kicad_pcb (KiCad board)
At the start: 0 parts

Commit message: First Draft of Power PCB
Parts:
- added B1: JST 2-PH, JSTPH2:JSTPH2, F.Cu at (228.4, 34.2)
- added C1: 10uF, Capacitor_SMD:C_1206_3216Metric_Pad1.33x1.80mm_HandSolder, F.Cu at (224.6, 39.6)
- added C10: 10u, Capacitor_SMD:C_1206_3216Metric_Pad1.33x1.80mm_HandSolder, F.Cu at (55.9, 137.1)
- added C11: 10u, Capacitor_SMD:C_1206_3216Metric_Pad1.33x1.80mm_HandSolder, F.Cu at (68.0, 137.1)
- added C12: 100n, Capacitor_SMD:C_1206_3216Metric_Pad1.33x1.80mm_HandSolder, F.Cu at (49.9, 137.3)
- added C13: 100n, Capacitor_SMD:C_1206_3216Metric_Pad1.33x1.80mm_HandSolder, F.Cu at (58.6, 133.8)
- added C14: 100n, Capacitor_SMD:C_1206_3216Metric_Pad1.33x1.80mm_HandSolder, F.Cu at (70.6, 133.8)
- added C15: 100n, Capacitor_SMD:C_1206_3216Metric_Pad1.33x1.80mm_HandSolder, F.Cu at (43.9, 134.0)
- added C16: 100n, Capacitor_SMD:C_1206_3216Metric_Pad1.33x1.80mm_HandSolder, F.Cu at (81.6, 118.2)
- added C17: 100n, Capacitor_SMD:C_1206_3216Metric_Pad1.33x1.80mm_HandSolder, F.Cu at (62.8, 112.2)
- added C18: 4.7uF, Capacitor_SMD:C_1206_3216Metric_Pad1.33x1.80mm_HandSolder, F.Cu at (91.3, 117.5)
- added C19: 4.7uF, Capacitor_SMD:C_1206_3216Metric_Pad1.33x1.80mm_HandSolder, F.Cu at (87.6, 120.9)
- added C2: 0.1uF, Capacitor_SMD:C_1206_3216Metric_Pad1.33x1.80mm_HandSolder, F.Cu at (211.4, 39.8)
- added C20: 27pF, Capacitor_SMD:C_1206_3216Metric_Pad1.33x1.80mm_HandSolder, F.Cu at (81.6, 124.9)
- added C21: 27pF, Capacitor_SMD:C_1206_3216Metric_Pad1.33x1.80mm_HandSolder, F.Cu at (106.1, 102.7)
- added C22: 10u, Capacitor_SMD:C_1206_3216Metric_Pad1.33x1.80mm_HandSolder, F.Cu at (81.6, 121.6)
- added C23: 10u, Capacitor_SMD:C_1206_3216Metric_Pad1.33x1.80mm_HandSolder, F.Cu at (49.9, 134.0)
- added C24: 10u, Capacitor_SMD:C_1206_3216Metric_Pad1.33x1.80mm_HandSolder, F.Cu at (62.0, 137.1)
- added C25: 10u, Capacitor_SMD:C_1206_3216Metric_Pad1.33x1.80mm_HandSolder, F.Cu at (64.6, 133.8)
- added C26: 100uF, Capacitor_SMD:C_1206_3216Metric_Pad1.33x1.80mm_HandSolder, F.Cu at (43.9, 137.3)
- added C3: 10uF, Capacitor_SMD:C_1206_3216Metric_Pad1.33x1.80mm_HandSolder, F.Cu at (214.2, 28.8)
- added C4: 2.2uF, Capacitor_SMD:C_1206_3216Metric_Pad1.33x1.80mm_HandSolder, F.Cu at (219.6, 51.8)
- added C5: 100uF, Capacitor_SMD:C_1206_3216Metric_Pad1.33x1.80mm_HandSolder, F.Cu at (219.6, 49.2)
- added C6: 10uF, Capacitor_SMD:C_1206_3216Metric_Pad1.33x1.80mm_HandSolder, F.Cu at (220.8, 32.8)
- added C7: 100n, Capacitor_SMD:C_1206_3216Metric_Pad1.33x1.80mm_HandSolder, F.Cu at (85.3, 75.6)
- added C8: 10u, Capacitor_SMD:C_1206_3216Metric_Pad1.33x1.80mm_HandSolder, F.Cu at (106.5, 45.6)
- added C9: 100n, Capacitor_SMD:C_1206_3216Metric_Pad1.33x1.80mm_HandSolder, F.Cu at (130.7, 33.3)
- added D1: Red, digikey-footprints:LED_5mm_Radial, F.Cu at (228.8, 45.0)
- added D2: Red, digikey-footprints:LED_5mm_Radial, F.Cu at (204.4, 52.3)
- added D3: Orange, digikey-footprints:LED_5mm_Radial, F.Cu at (204.0, 36.0)
- added D4: Green, digikey-footprints:LED_5mm_Radial, F.Cu at (204.0, 31.8)
- added D5: Green, digikey-footprints:LED_5mm_Radial, F.Cu at (74.6, 91.8)
- added D6: Red, digikey-footprints:LED_5mm_Radial, F.Cu at (102.4, 59.8)
- added J1: USB4125-GF-A_REVA2, USB4125-GF-A_REVA2:GCT_USB4125-GF-A_REVA2, F.Cu at (216.8, 23.0)
- added J2: SS-53000-001, SS-53000-001:STEWART_SS-53000-001, F.Cu at (113.1, 33.9)
- added J3: FFC3B07-20-T, FFC3B07-20-T:GCT_FFC3B07-20-T, F.Cu at (55.2, 92.7)
- added J4: Micro_SD_Card_Det, CM4IO:SDCARD_MOLEX_503398-1892, F.Cu at (89.8, 65.9)
- added J5: ARJM11D7-502-AB-EW2, ARJM11D7-502-AB-EW2:ARJM11D7502ABEW2, F.Cu at (98.6, 37.3)
- added J6: SS-52100-001, SS-52100-001:SS-52100-001, F.Cu at (66.1, 124.3)
- added J7: SS-52100-001, SS-52100-001:SS-52100-001, F.Cu at (47.2, 118.3)
- added J8: SS-52100-001, SS-52100-001:SS-52100-001, F.Cu at (75.8, 108.8)
- added J9: FFC3B07-20-T, FFC3B07-20-T:GCT_FFC3B07-20-T, F.Cu at (55.2, 105.8)
- added L1: 6.8uH, NRS5030T6R8MMGJ:NRS5030T6R8MMGJ, F.Cu at (222.0, 43.8)
- added Module1: ComputeModule4-CM4, CM4IO:Raspberry-Pi-4-Compute-Module, F.Cu at (45.1, 83.8)
- added Q1: MMUN2133LT1G, MMUN2133LT1G:SOT95P240X111-3N, F.Cu at (211.2, 43.4)
- added R1: 1.87M, Resistor_SMD:R_1206_3216Metric_Pad1.30x1.75mm_HandSolder, F.Cu at (219.4, 37.2)
- added R10: 15k, Resistor_SMD:R_1206_3216Metric_Pad1.30x1.75mm_HandSolder, F.Cu at (212.0, 31.2)
- added R11: 100k, Resistor_SMD:R_1206_3216Metric_Pad1.30x1.75mm_HandSolder, F.Cu at (209.3, 35.0)
- added R12: 1.0k, Resistor_SMD:R_1206_3216Metric_Pad1.30x1.75mm_HandSolder, F.Cu at (213.0, 35.0)
- added R13: 270k, Resistor_SMD:R_1206_3216Metric_Pad1.30x1.75mm_HandSolder, F.Cu at (219.2, 28.8)
- added R14: 1k, Resistor_SMD:R_1206_3216Metric_Pad1.30x1.75mm_HandSolder, F.Cu at (214.4, 51.8)
- added R15: 1k, Resistor_SMD:R_1206_3216Metric_Pad1.30x1.75mm_HandSolder, F.Cu at (112.5, 45.6)
- added R16: 12k 1%, Resistor_SMD:R_1206_3216Metric_Pad1.30x1.75mm_HandSolder, F.Cu at (106.5, 52.2)
- added R17: 1k, Resistor_SMD:R_1206_3216Metric_Pad1.30x1.75mm_HandSolder, F.Cu at (106.5, 49.0)
- added R18: 470R, Resistor_SMD:R_1206_3216Metric_Pad1.30x1.75mm_HandSolder, F.Cu at (112.4, 49.0)
- added R19: 470R, Resistor_SMD:R_1206_3216Metric_Pad1.30x1.75mm_HandSolder, F.Cu at (118.4, 48.9)
- added R2: 340k, Resistor_SMD:R_1206_3216Metric_Pad1.30x1.75mm_HandSolder, F.Cu at (219.4, 39.6)
- added R20: 36K 1%, Resistor_SMD:R_1206_3216Metric_Pad1.30x1.75mm_HandSolder, F.Cu at (76.6, 133.7)
- added R21: 36K 1%, Resistor_SMD:R_1206_3216Metric_Pad1.30x1.75mm_HandSolder, F.Cu at (81.6, 128.3)
- added R22: 12K 1%, Resistor_SMD:R_1206_3216Metric_Pad1.30x1.75mm_HandSolder, F.Cu at (73.9, 137.1)
- added R23: 15K 1%, Resistor_SMD:R_1206_3216Metric_Pad1.30x1.75mm_HandSolder, F.Cu at (97.3, 117.5)
- added R3: 5.1k, Resistor_SMD:R_1206_3216Metric_Pad1.30x1.75mm_HandSolder, F.Cu at (210.2, 25.0)
- added R4: 5.1k, Resistor_SMD:R_1206_3216Metric_Pad1.30x1.75mm_HandSolder, F.Cu at (223.5, 25.0)
- added R5: 200k, Resistor_SMD:R_1206_3216Metric_Pad1.30x1.75mm_HandSolder, F.Cu at (215.6, 38.4)
- added R6: 1k, Resistor_SMD:R_1206_3216Metric_Pad1.30x1.75mm_HandSolder, F.Cu at (211.2, 46.8)
- added R7: 1.87M, Resistor_SMD:R_1206_3216Metric_Pad1.30x1.75mm_HandSolder, F.Cu at (214.4, 49.2)
- added R8: 200k, Resistor_SMD:R_1206_3216Metric_Pad1.30x1.75mm_HandSolder, F.Cu at (209.0, 49.2)
- added R9: 100k, Resistor_SMD:R_1206_3216Metric_Pad1.30x1.75mm_HandSolder, F.Cu at (224.3, 28.8)
- added U1: TPS61090RSAR, TPS61090RSAR:QFN65P400X400X100-17N, F.Cu at (216.5, 44.0)
- added U2: MCP73871-2CCI_ML, digikey-footprints:QFN-20-1EP_4x4mm, F.Cu at (216.8, 33.5)
- added U3: 74LVC1G07, Package_TO_SOT_SMD:SOT-353_SC-70-5, F.Cu at (107.1, 61.4)
- added U4: RT9742VGJ5, Package_TO_SOT_SMD:SOT-23-5, F.Cu at (107.6, 57.3)
- added U5: RT9742ENGJ5, Package_TO_SOT_SMD:SOT-23-5, F.Cu at (112.0, 52.8)
- added U6: TPD4EUSB30, Package_SON:USON-10_2.5x1.0mm_P0.5mm, F.Cu at (89.7, 76.0)
- added U7: TPD4EUSB30, Package_SON:USON-10_2.5x1.0mm_P0.5mm, F.Cu at (129.1, 37.0)
- added U8: USB2504A-JT, USB2504A-JT:USB2504A-JT, F.Cu at (95.7, 108.5)
- added U9: AP22653W6-7, AP22653W6-7:SOT95P280X145-6N, F.Cu at (93.8, 121.4)
- added Y1: 24MHz, Crystal:Crystal_SMD_HC49-SD, F.Cu at (48.2, 129.2)
Routing:
- net VBUS: track 0.00 -> 40.9 mm, vias 0 -> 4
- net VBAT: track 0.00 -> 28.1 mm
- net Net-(D1-Pad2): track 0.00 -> 16.8 mm, vias 0 -> 2
- net Net-(D3-Pad1): track 0.00 -> 13.5 mm
- net Net-(D4-Pad1): track 0.00 -> 12.7 mm
- net /CM4/5v: track 0.00 -> 12.5 mm
- net Net-(B1-Pad2): track 0.00 -> 12.4 mm, vias 0 -> 2
- net Net-(D2-Pad1): track 0.00 -> 9.77 mm
- net Net-(R7-Pad2): track 0.00 -> 9.10 mm
- net Net-(J1-PadA5): track 0.00 -> 7.76 mm
- net Net-(J1-PadB5): track 0.00 -> 7.59 mm
- net Net-(R11-Pad1): track 0.00 -> 7.37 mm
- net Net-(R13-Pad1): track 0.00 -> 6.97 mm
- net GND: track 0.00 -> 6.52 mm, vias 0 -> 8
- net Net-(L1-Pad2): track 0.00 -> 5.34 mm
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- added copper zone on B.Cu, net GND
- added copper zone on F.Cu, net GND
Other:
- copper layers 0 -> 2
