File: kicad/customBoard/cm4.kicad_sch (KiCad schematic)
At the start: 20 parts, among them J2 SS-53000-001, J3 FFC3B07-20-T, J4 Micro_SD_Card_Det, J5 ARJM11D7-502-AB-EW2, U3 74LVC1G07, U4 RT9742VGJ5, U5 RT9742ENGJ5, U6 TPD4EUSB30, U7 TPD4EUSB30

Commit message: Save progress on USB
Connections:
- net 3.3v is gone; now on net +3V3: Module1.86 (+3.3v_(Output))
- net GND: no longer Module1.107 (GND), Module1.108 (GND), Module1.113 (GND), Module1.114 (GND), Module1.119 (GND), Module1.120 (GND), Module1.125 (GND), Module1.126 (GND), Module1.131 (GND), Module1.132 (GND), Module1.137 (GND), Module1.138 (GND), Module1.144 (GND), Module1.150 (GND), Module1.155 (GND), Module1.156 (GND), Module1.161 (GND), Module1.162 (GND), Module1.167 (GND), Module1.168 (GND), Module1.173 (GND), Module1.174 (GND), Module1.179 (GND), Module1.180 (GND), Module1.185 (GND), Module1.186 (GND), Module1.191 (GND), Module1.192 (GND), Module1.197 (GND), Module1.198 (GND)
- net HDMI0_CEC: no longer Module1.151 (HDMI0_CEC)
- net HDMI0_CK_N: no longer Module1.190 (HDMI0_CLK_N)
- net HDMI0_CK_P: no longer Module1.188 (HDMI0_CLK_P)
- net HDMI0_D0_N: no longer Module1.184 (HDMI0_TX0_N)
- net HDMI0_D0_P: no longer Module1.182 (HDMI0_TX0_P)
- net HDMI0_D1_N: no longer Module1.178 (HDMI0_TX1_N)
- net HDMI0_D1_P: no longer Module1.176 (HDMI0_TX1_P)
- net HDMI0_D2_N: no longer Module1.172 (HDMI0_TX2_N)
- net HDMI0_D2_P: no longer Module1.170 (HDMI0_TX2_P)
- net HDMI0_HOTPLUG: no longer Module1.153 (HDMI0_HOTPLUG)
- net HDMI0_SCL: no longer Module1.200 (HDMI0_SCL)
- net HDMI0_SDA: no longer Module1.199 (HDMI0_SDA)
- net HDMI1_CEC: no longer Module1.149 (HDMI1_CEC)
- net HDMI1_CK_N: no longer Module1.166 (HDMI1_CLK_N)
- net HDMI1_CK_P: no longer Module1.164 (HDMI1_CLK_P)
- net HDMI1_D0_N: no longer Module1.160 (HDMI1_TX0_N)
- net HDMI1_D0_P: no longer Module1.158 (HDMI1_TX0_P)
- net HDMI1_D1_N: no longer Module1.154 (HDMI1_TX1_N)
- net HDMI1_D1_P: no longer Module1.152 (HDMI1_TX1_P)
- net HDMI1_D2_N: no longer Module1.148 (HDMI1_TX2_N)
- net HDMI1_D2_P: no longer Module1.146 (HDMI1_TX2_P)
- net HDMI1_HOTPLUG: no longer Module1.143 (HDMI1_HOTPLUG)
- net HDMI1_SCL: no longer Module1.147 (HDMI1_SCL)
- net HDMI1_SDA: no longer Module1.145 (HDMI1_SDA)
- net TRD0_N: no longer U7.2 (D1-)
- net TRD0_P: no longer U7.1 (D1+)
- net TRD1_N: now also U7.2 (D1-)
- net TRD1_P: now also U7.1 (D1+)
- net USB2_N: no longer Module1.103 (USB2_N)
- net USB2_P: no longer Module1.105 (USB2_P)
Other:
- moved on the sheet: Module1B
Changed lines of the file:
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@@
   (junction (at 88.9 142.24) (diameter 0.9144) (color 0 0 0 0))
   (junction (at 110.49 173.99) (diameter 0.9144) (color 0 0 0 0))
+  (junction (at 111.76 43.18) (diameter 0.9144) (color 0 0 0 0))
+  (junction (at 111.76 45.72) (diameter 0.9144) (color 0 0 0 0))
   (junction (at 113.03 58.42) (diameter 0.9144) (color 0 0 0 0))
   (junction (at 113.03 68.58) (diameter 0.9144) (color 0 0 0 0))
@@
     (stroke (width 0) (type solid) (color 0 0 0 0))
   )
-  (wire (pts (xy 110.49 43.18) (xy 114.3 43.18))
+  (wire (pts (xy 110.49 43.18) (xy 111.76 43.18))
     (stroke (width 0) (type solid) (color 0 0 0 0))
   )
@@
   )
   (wire (pts (xy 110.49 173.99) (xy 123.19 173.99))
+    (stroke (width 0) (type solid) (color 0 0 0 0))
+  )
+  (wire (pts (xy 111.76 43.18) (xy 111.76 45.72))
+    (stroke (width 0) (type solid) (color 0 0 0 0))
+  )
+  (wire (pts (xy 111.76 43.18) (xy 114.3 43.18))
     (stroke (width 0) (type solid) (color 0 0 0 0))
   )
@@
     (effects (font (size 1.27 1.27)) (justify right bottom))
   )
-  (label "TRD0_P" (at 241.3 100.33 0)
-    (effects (font (size 1.27 1.27)) (justify left bottom))
-  )
-  (label "TRD0_N" (at 241.3 105.41 0)
+  (label "TRD1_P" (at 241.3 100.33 0)
+    (effects (font (size 1.27 1.27)) (justify left bottom))
+  )
+  (label "TRD1_N" (at 241.3 105.41 0)
     (effects (font (size 1.27 1.27)) (justify left bottom))
   )
@@
     (pin "9")
   )
-  (symbol (lib_id "CM4IO:ComputeModule4-CM4") (at -82.55 88.9 0) (mirror x) (unit 2)
+  (symbol (lib_id "CM4IO:ComputeModule4-CM4") (at -82.55 88.9 180) (unit 2)
     (in_bom yes) (on_board yes) (fields_autoplaced)
-    (property "Reference" "Module1" (id 0) (at 57.15 13.97 0))
-    (property "Value" "ComputeModule4-CM4" (id 1) (at 57.15 16.51 0))
-    (property "Footprint" "CM4IO:Raspberry-Pi-4-Compute-Module" (id 2) (at 59.69 62.23 0)
-      (effects (font (size 1.27 1.27)) hide)
-    )
-    (property "Datasheet" "" (id 3) (at 59.69 62.23 0)
-      (effects (font (size 1.27 1.27)) hide)
-    )
-    (property "Field4" "Hirose" (id 4) (at 57.15 19.05 0))
-    (property "Field5" "2x DF40C-100DS-0.4V" (id 5) (at 57.15 21.59 0))
+    (property "Reference" "Module1" (id 0) (at -222.25 13.97 0))
+    (property "Value" "ComputeModule4-CM4" (id 1) (at -222.25 16.51 0))
+    (property "Footprint" "CM4IO:Raspberry-Pi-4-Compute-Module" (id 2) (at -224.79 62.23 0)
+      (effects (font (size 1.27 1.27)) hide)
+    )
+    (property "Datasheet" "" (id 3) (at -224.79 62.23 0)
+      (effects (font (size 1.27 1.27)) hide)
+    )
+    (property "Field4" "Hirose" (id 4) (at -222.25 19.05 0))
+    (property "Field5" "2x DF40C-100DS-0.4V" (id 5) (at -222.25 21.59 0))
     (pin "101")
     (pin "102")

Commit message: Draft HDMI and more differential pairs
Parts:
- removed unit 2 of Module1
- added unit 2 of Module2
- renumbered Module1 to Module2
Connections:
- net GND: now also Module2.107 (GND), Module2.108 (GND), Module2.113 (GND), Module2.114 (GND), Module2.119 (GND), Module2.120 (GND), Module2.125 (GND), Module2.126 (GND), Module2.131 (GND), Module2.132 (GND), Module2.137 (GND), Module2.138 (GND), Module2.144 (GND), Module2.150 (GND), Module2.155 (GND), Module2.156 (GND), Module2.161 (GND), Module2.162 (GND), Module2.167 (GND), Module2.168 (GND), Module2.173 (GND), Module2.174 (GND), Module2.179 (GND), Module2.180 (GND), Module2.185 (GND), Module2.186 (GND), Module2.191 (GND), Module2.192 (GND), Module2.197 (GND), Module2.198 (GND)
- net HDMI0_CEC: now also Module2.151 (HDMI0_CEC)
- net HDMI0_CK_N: now also Module2.190 (HDMI0_CLK_N)
- net HDMI0_CK_P: now also Module2.188 (HDMI0_CLK_P)
- net HDMI0_D0_N: now also Module2.184 (HDMI0_TX0_N)
- net HDMI0_D0_P: now also Module2.182 (HDMI0_TX0_P)
- net HDMI0_D1_N: now also Module2.178 (HDMI0_TX1_N)
- net HDMI0_D1_P: now also Module2.176 (HDMI0_TX1_P)
- net HDMI0_D2_N: now also Module2.172 (HDMI0_TX2_N)
- net HDMI0_D2_P: now also Module2.170 (HDMI0_TX2_P)
- net HDMI0_HOTPLUG: now also Module2.153 (HDMI0_HOTPLUG)
- net HDMI0_SCL: now also Module2.200 (HDMI0_SCL)
- net HDMI0_SDA: now also Module2.199 (HDMI0_SDA)
- net HDMI1_CEC: now also Module2.149 (HDMI1_CEC)
- net HDMI1_CK_N: now also Module2.166 (HDMI1_CLK_N)
- net HDMI1_CK_P: now also Module2.164 (HDMI1_CLK_P)
- net HDMI1_D0_N: now also Module2.160 (HDMI1_TX0_N)
- net HDMI1_D0_P: now also Module2.158 (HDMI1_TX0_P)
- net HDMI1_D1_N: now also Module2.154 (HDMI1_TX1_N)
- net HDMI1_D1_P: now also Module2.152 (HDMI1_TX1_P)
- net HDMI1_D2_N: now also Module2.148 (HDMI1_TX2_N)
- net HDMI1_D2_P: now also Module2.146 (HDMI1_TX2_P)
- net HDMI1_HOTPLUG: now also Module2.143 (HDMI1_HOTPLUG)
- net HDMI1_SCL: now also Module2.147 (HDMI1_SCL)
- net HDMI1_SDA: now also Module2.145 (HDMI1_SDA)
- net USB2_N: now also Module2.103 (USB2_N)
- net USB2_P: now also Module2.105 (USB2_P)
Changed lines of the file:
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@@
   (symbol (lib_id "power:GND") (at 25.4 152.4 0) (unit 1)
     (in_bom yes) (on_board yes)
-    (property "Reference" "#PWR035" (id 0) (at 25.4 158.75 0)
+    (property "Reference" "#PWR034" (id 0) (at 25.4 158.75 0)
       (effects (font (size 1.27 1.27)) hide)
     )
@@
   (symbol (lib_id "power:GND") (at 25.4 180.34 0) (unit 1)
     (in_bom yes) (on_board yes)
-    (property "Reference" "#PWR037" (id 0) (at 25.4 186.69 0)
+    (property "Reference" "#PWR035" (id 0) (at 25.4 186.69 0)
       (effects (font (size 1.27 1.27)) hide)
     )
@@
   (symbol (lib_id "power:GND") (at 105.41 180.34 0) (unit 1)
     (in_bom yes) (on_board yes)
-    (property "Reference" "#PWR034" (id 0) (at 105.41 186.69 0)
+    (property "Reference" "#PWR037" (id 0) (at 105.41 186.69 0)
       (effects (font (size 1.27 1.27)) hide)
     )
@@
     (pin "9")
   )
-  (symbol (lib_id "CM4IO:ComputeModule4-CM4") (at -82.55 88.9 180) (unit 2)
-    (in_bom yes) (on_board yes) (fields_autoplaced)
-    (property "Reference" "Module1" (id 0) (at -222.25 13.97 0))
-    (property "Value" "ComputeModule4-CM4" (id 1) (at -222.25 16.51 0))
-    (property "Footprint" "CM4IO:Raspberry-Pi-4-Compute-Module" (id 2) (at -224.79 62.23 0)
-      (effects (font (size 1.27 1.27)) hide)
-    )
-    (property "Datasheet" "" (id 3) (at -224.79 62.23 0)
-      (effects (font (size 1.27 1.27)) hide)
-    )
-    (property "Field4" "Hirose" (id 4) (at -222.25 19.05 0))
-    (property "Field5" "2x DF40C-100DS-0.4V" (id 5) (at -222.25 21.59 0))
+  (symbol (lib_id "CM4IO:ComputeModule4-CM4") (at -82.55 88.9 0) (mirror x) (unit 2)
+    (in_bom yes) (on_board yes) (fields_autoplaced)
+    (property "Reference" "Module2" (id 0) (at 57.15 13.97 0))
+    (property "Value" "ComputeModule4-CM4" (id 1) (at 57.15 16.51 0))
+    (property "Footprint" "CM4IO:Raspberry-Pi-4-Compute-Module" (id 2) (at 59.69 62.23 0)
+      (effects (font (size 1.27 1.27)) hide)
+    )
+    (property "Datasheet" "" (id 3) (at 59.69 62.23 0)
+      (effects (font (size 1.27 1.27)) hide)
+    )
+    (property "Field4" "Hirose" (id 4) (at 57.15 19.05 0))
+    (property "Field5" "2x DF40C-100DS-0.4V" (id 5) (at 57.15 21.59 0))
     (pin "101")
     (pin "102")
@@
   (symbol (lib_id "CM4IO:ComputeModule4-CM4") (at 147.32 93.98 0) (mirror x) (unit 1)
     (in_bom yes) (on_board yes) (fields_autoplaced)
-    (property "Reference" "Module1" (id 0) (at 144.78 13.97 0))
+    (property "Reference" "Module2" (id 0) (at 144.78 13.97 0))
     (property "Value" "ComputeModule4-CM4" (id 1) (at 144.78 16.51 0))
     (property "Footprint" "CM4IO:Raspberry-Pi-4-Compute-Module" (id 2) (at 289.56 67.31 0)

Commit message: Updates based on meeting with Dr. Jordan
Everything should be good to go now, next up is generating a bill of materials (making sure everything is in stock), and generating gerbers
Parts:
- D5, D6: footprint digikey-footprints:LED_5mm_Radial -> LED_SMD:LED_1206_3216Metric_Pad1.42x1.75mm_HandSolder
- renumbered J2 to J3, J3 to J4, J4 to J5, J5 to J6, Module2 to Module1

Commit message: Generate BOM
Clean up all the part data and add manufacturer's numbers for ordering
Parts:
- C7: value 100n -> 0.1uF; Part Description 0.1uF 10% 16V Ceramic Capacitor X7R 0402 (1005 Metric) -> (none); manf# (none) -> CL31B104KBCNFNC
- C8: value 10u -> 10uF; manf# (none) -> CL31B106MOHNNNE
- C9: value 100n -> 0.1uF; manf# (none) -> CL31B104KBCNFNC
- D5: manf# (none) -> 150120GS75000
- D6: manf# (none) -> 156120RS75300
- J3: MANUFACTURER BelFuse -> (none); MAXIMUM_PACKAGE_HEIGHT 6.18 mm -> (none); PARTREV A0 -> (none); STANDARD Manufacturer Recommendations -> (none); manf# (none) -> SS-53000-001
- J4: MANUFACTURER GCT -> (none); MAXIMUM_PACKAGE_HEIGHT 2.5mm -> (none); PARTREV A -> (none); STANDARD Manufacturer Recommendations -> (none); manf# (none) -> FFC3B07-20-T
- J5: manf# (none) -> 5033981892
- J6: Height 13.8 -> (none); Manufacturer_Name ABRACON -> (none); Manufacturer_Part_Number ARJM11D7-502-AB-EW2 -> (none); Mouser Part Number 815-RJM11D7502ABEW2 -> (none); Mouser Price/Stock https://www.mouser.co.uk/ProductDetail/ABRACON/ARJM11D7-502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 -> (none); manf# (none) -> ARJM11D7-502-AB-EW2
- R17, R19: value 1k -> 1K; manf# (none) -> RC1206FR-071KL
- R18: value 12k 1% -> 12K 1%; manf# (none) -> RC1206FR-0712KL
- R20, R21: manf# (none) -> RC1206FR-07470RL
- U3: manf# (none) -> 74LVC1G07SE-7
- U4: Part Description Power Switch/Driver 1:1 N-Channel 1A TSOT-23-5 -> (none); manf# (none) -> RT9742VGJ5
- U5: Part Description Power Switch/Driver 1:1 N-Channel 1A TSOT-23-5 -> (none); manf# (none) -> RT9742ENGJ5
- U6, U7: manf# (none) -> TPD4EUSB30DQAR
Changed lines of the file:
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@@
     (in_bom yes) (on_board yes)
     (property "Reference" "R17" (id 0) (at 186.69 121.92 90))
-    (property "Value" "1k" (id 1) (at 186.69 124.46 90))
+    (property "Value" "1K" (id 1) (at 186.69 124.46 90))
     (property "Footprint" "Resistor_SMD:R_1206_3216Metric_Pad1.30x1.75mm_HandSolder" (id 2) (at 186.69 126.238 90)
       (effects (font (size 1.27 1.27)) hide)
@@
       (effects (font (size 1.27 1.27)) hide)
     )
+    (property "manf#" "RC1206FR-071KL" (id 4) (at 186.69 124.46 0)
+      (effects (font (size 1.27 1.27)) hide)
+    )
     (pin "1")
     (pin "2")
@@
     (in_bom yes) (on_board yes)
     (property "Reference" "R18" (id 0) (at 193.04 46.99 90))
-    (property "Value" "12k 1%" (id 1) (at 198.12 46.99 90))
+    (property "Value" "12K 1%" (id 1) (at 198.12 46.99 90))
     (property "Footprint" "Resistor_SMD:R_1206_3216Metric_Pad1.30x1.75mm_HandSolder" (id 2) (at 197.358 46.99 90)
       (effects (font (size 1.27 1.27)) hide)
@@
       (effects (font (size 1.27 1.27)) hide)
     )
+    (property "manf#" "RC1206FR-0712KL" (id 4) (at 195.58 46.99 0)
+      (effects (font (size 1.27 1.27)) hide)
+    )
     (pin "1")
     (pin "2")
@@
     (in_bom yes) (on_board yes)
     (property "Reference" "R19" (id 0) (at 204.47 27.94 90))
-    (property "Value" "1k" (id 1) (at 204.47 30.48 90))
+    (property "Value" "1K" (id 1) (at 204.47 30.48 90))
     (property "Footprint" "Resistor_SMD:R_1206_3216Metric_Pad1.30x1.75mm_HandSolder" (id 2) (at 204.47 32.258 90)
       (effects (font (size 1.27 1.27)) hide)
     )
     (property "Datasheet" "~" (id 3) (at 204.47 30.48 0)
+      (effects (font (size 1.27 1.27)) hide)
+    )
+    (property "manf#" "RC1206FR-071KL" (id 4) (at 204.47 30.48 0)
       (effects (font (size 1.27 1.27)) hide)
     )
@@
       (effects (font (size 1.27 1.27)) hide)
     )
+    (property "manf#" "RC1206FR-07470RL" (id 4) (at 220.98 71.12 0)
+      (effects (font (size 1.27 1.27)) hide)
+    )
     (pin "1")
     (pin "2")
@@
       (effects (font (size 1.27 1.27)) hide)
     )
+    (property "manf#" "RC1206FR-07470RL" (id 4) (at 220.98 76.2 0)
+      (effects (font (size 1.27 1.27)) hide)
+    )
     (pin "1")
     (pin "2")
@@
       (effects (font (size 1.27 1.27)) hide)
     )
+    (property "manf#" "150120GS75000" (id 4) (at 196.85 124.46 0)
+      (effects (font (size 1.27 1.27)) hide)
+    )
     (pin "1")
     (pin "2")
@@
       (effects (font (size 1.27 1.27)) hide)
     )
+    (property "manf#" "156120RS75300" (id 4) (at 214.63 30.48 0)
+      (effects (font (size 1.27 1.27)) hide)
+    )
     (pin "1")
     (pin "2")
@@
       (effects (font (size 1.27 1.27)) (justify left))
     )
-    (property "Value" "100n" (id 1) (at 204.851 142.113 0)
+    (property "Value" "0.1uF" (id 1) (at 204.851 142.113 0)
       (effects (font (size 1.27 1.27)) (justify left))
     )
@@
       (effects (font (size 1.27 1.27)) hide)
     )
-    (property "Part Description" "	0.1uF 10% 16V Ceramic Capacitor X7R 0402 (1005 Metric)" (id 8) (at 201.93 140.97 0)
-      (effects (font (size 1.27 1.27)) hide)
-    )
     (property "Field8" "110091611" (id 9) (at 201.93 140.97 0)
       (effects (font (size 1.27 1.27)) hide)
     )
+    (property "manf#" "CL31B104KBCNFNC" (id 10) (at 201.93 140.97 0)
+      (effects (font (size 1.27 1.27)) hide)
+    )
     (pin "1")
     (pin "2")
@@
       (effects (font (size 1.27 1.27)) (justify left))
     )
-    (property "Value" "10u" (id 1) (at 226.06 41.2749 0)
+    (property "Value" "10uF" (id 1) (at 226.06 41.2749 0)
       (effects (font (size 1.27 1.27)) (justify left))
     )
@@
       (effects (font (size 1.27 1.27)) hide)
     )
+    (property "manf#" "CL31B106MOHNNNE" (id 4) (at 222.25 39.37 0)
+      (effects (font (size 1.27 1.27)) hide)
+    )
     (pin "1")
     (pin "2")
@@
     (in_bom yes) (on_board yes) (fields_autoplaced)
     (property "Reference" "C9" (id 0) (at 276.86 66.04 90))
-    (property "Value" "100n" (id 1) (at 276.86 68.58 90))
+    (property "Value" "0.1uF" (id 1) (at 276.86 68.58 90))
     (property "Footprint" "Capacitor_SMD:C_1206_3216Metric_Pad1.33x1.80mm_HandSolder" (id 2) (at 280.67 71.4248 0)
       (effects (font (size 1.27 1.27)) hide)
@@
       (effects (font (size 1.27 1.27)) hide)
     )
+    (property "manf#" "CL31B104KBCNFNC" (id 4) (at 276.86 72.39 0)
+      (effects (font (size 1.27 1.27)) hide)
+    )
     (pin "1")
     (pin "2")
@@
     )
     (property "Datasheet" "http://www.ti.com/lit/sg/scyt129e/scyt129e.pdf" (id 3) (at 186.69 30.48 0)
+      (effects (font (size 1.27 1.27)) hide)
+    )
+    (property "manf#" "74LVC1G07SE-7" (id 4) (at 186.69 30.48 0)
       (effects (font (size 1.27 1.27)) hide)
     )
@@
       (effects (font (size 1.27 1.27)) hide)
     )
-    (property "Part Description" "	Power Switch/Driver 1:1 N-Channel 1A TSOT-23-5" (id 9) (at 207.01 53.34 0)
+    (property "manf#" "RT9742VGJ5" (id 10) (at 207.01 53.34 0)
       (effects (font (size 1.27 1.27)) hide)
     )
@@
       (effects (font (size 1.27 1.27)) hide)
     )
-    (property "Part Description" "	Power Switch/Driver 1:1 N-Channel 1A TSOT-23-5" (id 9) (at 215.9 144.78 0)
+    (property "manf#" "RT9742ENGJ5" (id 10) (at 215.9 144.78 0)
       (effects (font (size 1.27 1.27)) hide)
     )
@@
     )
     (property "Datasheet" "http://www.ti.com/lit/ds/symlink/tpd2eusb30a.pdf" (id 3) (at 217.17 102.87 0)
+      (effects (font (size 1.27 1.27)) hide)
+    )
+    (property "manf#" "TPD4EUSB30DQAR" (id 4) (at 217.17 102.87 0)
       (effects (font (size 1.27 1.27)) hide)
     )
@@
       (effects (font (size 1.27 1.27)) hide)
     )
+    (property "manf#" "TPD4EUSB30DQAR" (id 4) (at 261.62 102.87 0)
+      (effects (font (size 1.27 1.27)) hide)
+    )
     (pin "1")
     (pin "10")
@@
       (effects (font (size 1.27 1.27)) (justify left) hide)
     )
-    (property "Description" "Modular Connectors / Ethernet Connectors RJ45 JACK W/MAG 1000Base-T" (id 4) (at 229.87 81.28 0)
-      (effects (font (size 1.27 1.27)) (justify left) hide)
-    )
-    (property "Height" "13.8" (id 5) (at 229.87 78.74 0)
-      (effects (font (size 1.27 1.27)) (justify left) hide)
-    )
-    (property "Mouser Part Number" "815-RJM11D7502ABEW2" (id 6) (at 229.87 76.2 0)
-      (effects (font (size 1.27 1.27)) (justify left) hide)
-    )
-    (property "Mouser Price/Stock" "https://www.mouser.co.uk/ProductDetail/ABRACON/ARJM11D7-502-AB-EW2?qs=YCa%2FAAYMW02O0E7mrqREQQ%3D%3D" (id 7) (at 229.87 73.66 0)
-      (effects (font (size 1.27 1.27)) (justify left) hide)
-    )
-    (property "Manufacturer_Name" "ABRACON" (id 8) (at 229.87 71.12 0)
-      (effects (font (size 1.27 1.27)) (justify left) hide)
-    )
-    (property "Manufacturer_Part_Number" "ARJM11D7-502-AB-EW2" (id 9) (at 229.87 68.58 0)
-      (effects (font (size 1.27 1.27)) (justify left) hide)
+    (property "manf#" "ARJM11D7-502-AB-EW2" (id 4) (at 264.16 83.82 0)
+      (effects (font (size 1.27 1.27)) hide)
     )
     (pin "1")
@@
       (effects (font (size 1.27 1.27)) (justify left bottom) hide)
     )
-    (property "PARTREV" "A" (id 4) (at 138.43 185.42 0)
-      (effects (font (size 1.27 1.27)) (justify left bottom) hide)
-    )
-    (property "STANDARD" "Manufacturer Recommendations" (id 5) (at 138.43 185.42 0)
-      (effects (font (size 1.27 1.27)) (justify left bottom) hide)
-    )
-    (property "MAXIMUM_PACKAGE_HEIGHT" "2.5mm" (id 6) (at 138.43 185.42 0)
-      (effects (font (size 1.27 1.27)) (justify left bottom) hide)
-    )
-    (property "MANUFACTURER" "GCT" (id 7) (at 138.43 185.42 0)
-      (effects (font (size 1.27 1.27)) (justify left bottom) hide)
+    (property "manf#" "FFC3B07-20-T" (id 4) (at 138.43 185.42 0)
+      (effects (font (size 1.27 1.27)) hide)
     )
     (pin "1")
@@
       (effects (font (size 1.27 1.27)) (justify left bottom) hide)
     )
-    (property "PARTREV" "A0" (id 4) (at 55.88 185.42 0)
-      (effects (font (size 1.27 1.27)) (justify left bottom) hide)
-    )
-    (property "STANDARD" "Manufacturer Recommendations" (id 5) (at 55.88 185.42 0)
-      (effects (font (size 1.27 1.27)) (justify left bottom) hide)
-    )
-    (property "MAXIMUM_PACKAGE_HEIGHT" "6.18 mm" (id 6) (at 55.88 185.42 0)
-      (effects (font (size 1.27 1.27)) (justify left bottom) hide)
-    )
-    (property "MANUFACTURER" "BelFuse" (id 7) (at 55.88 185.42 0)
-      (effects (font (size 1.27 1.27)) (justify left bottom) hide)
+    (property "manf#" "SS-53000-001" (id 4) (at 55.88 185.42 0)
+      (effects (font (size 1.27 1.27)) hide)
     )
     (pin "1")
@@
       (effects (font (size 1.27 1.27)) hide)
     )
+    (property "manf#" "5033981892" (id 4) (at 261.62 38.1 0)
+      (effects (font (size 1.27 1.27)) hide)
+    )
